File: CareMate/CareMate.sch (KiCad schematic (older format))
At the start: 19 parts, among them J1 Barrel_Jack_MountingPin, J2 Conn_01x16, J3 Conn_01x03, J4 Conn_01x03, J5 Conn_01x06, J6 Conn_01x03, J7 Conn_01x03, J8 Conn_01x02, U1 L7805, U2 LM386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

Commit message: Began assigning footprints, created new ones
Parts:
- J2: footprint (none) -> Additional Libraries:16PinConnector
- J3, J4, J6, J7: footprint (none) -> Additional Libraries:3PinConnector
- U3: symbol CareMate_Library:Elechouse_V3 -> CareMate-rescue:Elechouse_V3-CareMate_Library
- U4: footprint MODULE_ESP32-DEVKITC-32D -> ESP32:MODULE_ESP32-DEVKITC-32D
Changed lines of the file:
@@
 F 0 "U4" H 9450 3267 50  0000 C CNN
 F 1 "ESP32-DEVKITC-32D" H 9450 3176 50  0000 C CNN
-F 2 "MODULE_ESP32-DEVKITC-32D" H 9450 2100 50  0001 L BNN
+F 2 "ESP32:MODULE_ESP32-DEVKITC-32D" H 9450 2100 50  0001 L BNN
 F 3 "" H 9450 2100 50  0001 L BNN
 F 4 "ESP32-DEVKITC-32D" H 9450 2100 50  0001 L BNN "MP"
@@
 $EndComp
 $Comp
-L CareMate_Library:Elechouse_V3 U3
+L CareMate-rescue:Elechouse_V3-CareMate_Library U3
 U 1 1 608EC375
 P 5900 950
@@
 F 0 "J7" V 8622 4580 50  0000 L CNN
 F 1 "Conn_01x03" V 8713 4580 50  0000 L CNN
-F 2 "" H 8750 4400 50  0001 C CNN
+F 2 "Additional Libraries:3PinConnector" H 8750 4400 50  0001 C CNN
 F 3 "~" H 8750 4400 50  0001 C CNN
 	1    8750 4400
@@
 F 0 "J3" V 4922 5830 50  0000 L CNN
 F 1 "Conn_01x03" V 5013 5830 50  0000 L CNN
-F 2 "" H 5050 5650 50  0001 C CNN
+F 2 "Additional Libraries:3PinConnector" H 5050 5650 50  0001 C CNN
 F 3 "~" H 5050 5650 50  0001 C CNN
 	1    5050 5650
@@
 F 0 "J2" V 4900 5250 50  0000 C CNN
 F 1 "Conn_01x16" V 4800 5300 50  0000 C CNN
-F 2 "" H 5000 4250 50  0001 C CNN
+F 2 "Additional Libraries:16PinConnector" H 5000 4250 50  0001 C CNN
 F 3 "~" H 5000 4250 50  0001 C CNN
 	1    5000 4250
@@
 F 0 "J4" V 6722 5930 50  0000 L CNN
 F 1 "Conn_01x03" V 6813 5930 50  0000 L CNN
-F 2 "" H 6850 5750 50  0001 C CNN
+F 2 "Additional Libraries:3PinConnector" H 6850 5750 50  0001 C CNN
 F 3 "~" H 6850 5750 50  0001 C CNN
 	1    6850 5750
@@
 F 0 "J6" V 7572 5930 50  0000 L CNN
 F 1 "Conn_01x03" V 7663 5930 50  0000 L CNN
-F 2 "" H 7700 5750 50  0001 C CNN
+F 2 "Additional Libraries:3PinConnector" H 7700 5750 50  0001 C CNN
 F 3 "~" H 7700 5750 50  0001 C CNN
 	1    7700 5750

Commit message: Updated Footprints
Parts:
- J8: footprint (none) -> Additional Libraries:JST_B2B-PH-K-S(LF)(SN)
Changed lines of the file:
@@
 F 0 "J8" V 10364 4212 50  0000 R CNN
 F 1 "Conn_01x02" V 10273 4212 50  0000 R CNN
-F 2 "" H 10400 4400 50  0001 C CNN
+F 2 "Additional Libraries:JST_B2B-PH-K-S(LF)(SN)" H 10400 4400 50  0001 C CNN
 F 3 "~" H 10400 4400 50  0001 C CNN
 	1    10400 4400

Commit message: Finished assigning footprints and generated first netlist
Parts:
- C1, C2, C3, C4: footprint (none) -> Capacitor_SMD:C_0603_1608Metric_Pad1.05x0.95mm_HandSolder
- C5: footprint (none) -> Additional Libraries:CAPC3216X190N
- J1: footprint (none) -> Connector_BarrelJack:BarrelJack_Horizontal
- J5: footprint (none) -> Additional Libraries:SD_Card_Reader
- R1, R2: footprint (none) -> Resistor_SMD:R_0603_1608Metric_Pad1.05x0.95mm_HandSolder
- U1: footprint (none) -> Additional Libraries:L7805
- U2: footprint (none) -> Additional Libraries:LM386N
- U3: footprint (none) -> Additional Libraries:ElechouseV3
Changed lines of the file:
@@
 F 0 "U3" H 6125 1065 50  0000 C CNN
 F 1 "Elechouse_V3" H 6125 974 50  0000 C CNN
-F 2 "" H 5900 950 50  0001 C CNN
+F 2 "Additional Libraries:ElechouseV3" H 5900 950 50  0001 C CNN
 F 3 "" H 5900 950 50  0001 C CNN
 	1    5900 950
@@
 F 0 "U2" H 3344 1996 50  0000 L CNN
 F 1 "LM386" H 3344 1905 50  0000 L CNN
-F 2 "" H 3100 2050 50  0001 C CNN
+F 2 "Additional Libraries:LM386N" H 3100 2050 50  0001 C CNN
 F 3 "http://www.ti.com/lit/ds/symlink/lm386.pdf" H 3200 2150 50  0001 C CNN
 	1    3000 1950
@@
 F 0 "R1" V 3150 2500 50  0000 C CNN
 F 1 "1.2k" V 3250 2500 50  0000 C CNN
-F 2 "" V 3180 2500 50  0001 C CNN
+F 2 "Resistor_SMD:R_0603_1608Metric_Pad1.05x0.95mm_HandSolder" V 3180 2500 50  0001 C CNN
 F 3 "~" H 3250 2500 50  0001 C CNN
 	1    3250 2500
@@
 F 0 "C3" V 3371 2500 50  0000 C CNN
 F 1 "10uF" V 3462 2500 50  0000 C CNN
-F 2 "" H 3600 2500 50  0001 C CNN
+F 2 "Capacitor_SMD:C_0603_1608Metric_Pad1.05x0.95mm_HandSolder" H 3600 2500 50  0001 C CNN
 F 3 "~" H 3600 2500 50  0001 C CNN
 	1    3600 2500
@@
 F 0 "C5" V 3921 1950 50  0000 C CNN
 F 1 "250uF" V 4012 1950 50  0000 C CNN
-F 2 "" H 4150 1950 50  0001 C CNN
+F 2 "Additional Libraries:CAPC3216X190N" H 4150 1950 50  0001 C CNN
 F 3 "~" H 4150 1950 50  0001 C CNN
 	1    4150 1950
@@
 F 0 "R2" V 3850 2150 50  0000 C CNN
 F 1 "10" V 3950 2150 50  0000 C CNN
-F 2 "" V 3880 2150 50  0001 C CNN
+F 2 "Resistor_SMD:R_0603_1608Metric_Pad1.05x0.95mm_HandSolder" V 3880 2150 50  0001 C CNN
 F 3 "~" H 3950 2150 50  0001 C CNN
 	1    3950 2150
@@
 F 0 "J1" H 3007 4367 50  0000 C CNN
 F 1 "Barrel_Jack_MountingPin" H 3007 4276 50  0000 C CNN
-F 2 "" H 3000 4010 50  0001 C CNN
+F 2 "Connector_BarrelJack:BarrelJack_Horizontal" H 3000 4010 50  0001 C CNN
 F 3 "~" H 3000 4010 50  0001 C CNN
 	1    2950 4050
@@
 F 0 "U1" H 2850 5792 50  0000 C CNN
 F 1 "L7805" H 2850 5701 50  0000 C CNN
-F 2 "" H 2875 5400 50  0001 L CIN
+F 2 "Additional Libraries:L7805" H 2875 5400 50  0001 L CIN
 F 3 "http://www.st.com/content/ccc/resource/technical/document/datasheet/41/4f/b3/b0/12/d4/47/88/CD00000444.pdf/files/CD00000444.pdf/jcr:content/translations/en.CD00000444.pdf" H 2850 5500 50  0001 C CNN
 	1    2850 5550
@@
 F 0 "C1" H 2008 5654 50  0000 R CNN
 F 1 "0.33uF" H 2008 5745 50  0000 R CNN
-F 2 "" H 2100 5700 50  0001 C CNN
+F 2 "Capacitor_SMD:C_0603_1608Metric_Pad1.05x0.95mm_HandSolder" H 2100 5700 50  0001 C CNN
 F 3 "~" H 2100 5700 50  0001 C CNN
 	1    2100 5700
@@
 F 0 "C2" H 3458 5654 50  0000 R CNN
 F 1 "0.1uF" H 3458 5745 50  0000 R CNN
-F 2 "" H 3550 5700 50  0001 C CNN
+F 2 "Capacitor_SMD:C_0603_1608Metric_Pad1.05x0.95mm_HandSolder" H 3550 5700 50  0001 C CNN
 F 3 "~" H 3550 5700 50  0001 C CNN
 	1    3550 5700
@@
 F 0 "J5" V 6972 4630 50  0000 L CNN
 F 1 "Conn_01x06" V 7063 4630 50  0000 L CNN
-F 2 "" H 7100 4350 50  0001 C CNN
+F 2 "Additional Libraries:SD_Card_Reader" H 7100 4350 50  0001 C CNN
 F 3 "~" H 7100 4350 50  0001 C CNN
 	1    7100 4350
@@
 F 0 "C4" H 3750 2600 50  0000 C CNN
 F 1 ".05uF" H 3750 2500 50  0000 C CNN
-F 2 "" H 3950 2500 50  0001 C CNN
+F 2 "Capacitor_SMD:C_0603_1608Metric_Pad1.05x0.95mm_HandSolder" H 3950 2500 50  0001 C CNN
 F 3 "~" H 3950 2500 50  0001 C CNN
 	1    3950 2500

Commit message: generated PCB and loaded netlist
Parts:
- J3, J4, J6, J7: footprint Additional Libraries:3PinConnector -> Additional Libraries:3PinConnector_Official
Changed lines of the file:
@@
 F 0 "J7" V 8622 4580 50  0000 L CNN
 F 1 "Conn_01x03" V 8713 4580 50  0000 L CNN
-F 2 "Additional Libraries:3PinConnector" H 8750 4400 50  0001 C CNN
+F 2 "Additional Libraries:3PinConnector_Official" H 8750 4400 50  0001 C CNN
 F 3 "~" H 8750 4400 50  0001 C CNN
 	1    8750 4400
@@
 F 0 "J3" V 4922 5830 50  0000 L CNN
 F 1 "Conn_01x03" V 5013 5830 50  0000 L CNN
-F 2 "Additional Libraries:3PinConnector" H 5050 5650 50  0001 C CNN
+F 2 "Additional Libraries:3PinConnector_Official" H 5050 5650 50  0001 C CNN
 F 3 "~" H 5050 5650 50  0001 C CNN
 	1    5050 5650
@@
 F 0 "J4" V 6722 5930 50  0000 L CNN
 F 1 "Conn_01x03" V 6813 5930 50  0000 L CNN
-F 2 "Additional Libraries:3PinConnector" H 6850 5750 50  0001 C CNN
+F 2 "Additional Libraries:3PinConnector_Official" H 6850 5750 50  0001 C CNN
 F 3 "~" H 6850 5750 50  0001 C CNN
 	1    6850 5750
@@
 F 0 "J6" V 7572 5930 50  0000 L CNN
 F 1 "Conn_01x03" V 7663 5930 50  0000 L CNN
-F 2 "Additional Libraries:3PinConnector" H 7700 5750 50  0001 C CNN
+F 2 "Additional Libraries:3PinConnector_Official" H 7700 5750 50  0001 C CNN
 F 3 "~" H 7700 5750 50  0001 C CNN
 	1    7700 5750
